File: data.kicad_sch (KiCad schematic)
At the start: 33 parts, among them J1 Conn_01x11_Pin, J3 Conn_01x10_Pin, J6 GSB1C41110SSHR, U3 FT232H, U5 93LCxxB, Y1 ECS-120-8-36-CKM-TR3

Commit message: rev 3
Parts:
- removed J1: Conn_01x11_Pin, Connector_PinHeader_2.54mm:PinHeader_1x11_P2.54mm_Vertical, symbol Connector:Conn_01x11_Pin
- removed J3: Conn_01x10_Pin, Connector_PinHeader_2.54mm:PinHeader_1x10_P2.54mm_Vertical, symbol Connector:Conn_01x10_Pin
