File: tayloe.kicad_sch (KiCad schematic)
At the start: 55 parts, among them IC1 INA163UA_2K5, IC2 INA163UA_2K5, J2 SJ3-35063B, J4 Conn_01x02_Pin, U1 PI3B3253LEX, U2 SN74AC74PWR, U4 AP2112K-3.3, U6 Si5351A-B-GT, U7 ADP7182AUJZ-5.0, Y2 ABM8G-25.000MHZ-4Y-T3

Commit message: whatever
Parts:
- C12: value 47p -> 47u
Changed lines of the file:
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@@
 			)
 		)
-		(property "Value" "47p"
+		(property "Value" "47u"
 			(at 36.83 125.73 0)
 			(effects

Commit message: rev 2
Parts:
- removed IC1, IC2: INA163UA_2K5, Package_SO:SOIC-14_3.9x8.7mm_P1.27mm, symbol tayloe:INA163UA_2K5
- removed R12, R13, R14, R15, R22: 0, Resistor_SMD:R_1206_3216Metric_Pad1.30x1.75mm_HandSolder, symbol Device:R_Small
- added C45: 0.33u, Capacitor_SMD:C_0603_1608Metric, symbol Device:C_Small
- added C46: 0.1u, Capacitor_SMD:C_0603_1608Metric, symbol Device:C_Small
- added IC1, IC2: INA828IDR, Package_SO:SOIC-8_3.9x4.9mm_P1.27mm, symbol tayloe:INA828IDR
- added R23, R24, R25: 47k, Resistor_SMD:R_0603_1608Metric, symbol Device:R_Small
- added R3, R4: 10k, Resistor_SMD:R_0603_1608Metric, symbol Device:R_Small
- added U8: L78L08_SO8, Package_SO:SOIC-8_3.9x4.9mm_P1.27mm, symbol Regulator_Linear:L78L08_SO8
- C1, C10, C11, C2, C31, C32, C33, C34, C35, C36, C37, C40, C41, C43, C44, C7, C8, C9: footprint Capacitor_SMD:C_1206_3216Metric_Pad1.33x1.80mm_HandSolder -> Capacitor_SMD:C_0603_1608Metric
- C12: Mouser Part (none) -> 710-865080342006
- C3, C4, C5, C6: footprint Capacitor_SMD:C_1206_3216Metric_Pad1.33x1.80mm_HandSolder -> Capacitor_SMD:C_0603_1608Metric; Mouser Part (none) -> 603-CC603JRX7R8BB683
- C38, C39: value 0.47u -> 0.1u; footprint Capacitor_SMD:C_1206_3216Metric_Pad1.33x1.80mm_HandSolder -> Capacitor_SMD:C_0603_1608Metric
- FB4: footprint Inductor_SMD:L_1206_3216Metric_Pad1.22x1.90mm_HandSolder -> Inductor_SMD:L_0603_1608Metric; Mouser Part (none) -> 81-BLM18HK601SN1D
- L1, L2: footprint Inductor_SMD:L_1206_3216Metric_Pad1.42x1.75mm_HandSolder -> Inductor_SMD:L_0603_1608Metric
- R1, R2: value 100 -> 330; footprint Resistor_SMD:R_1206_3216Metric_Pad1.30x1.75mm_HandSolder -> Resistor_SMD:R_0603_1608Metric; Mouser Part (none) -> 603-RT0603DRE07330RL
- R16: value 0 -> 47k; footprint Resistor_SMD:R_1206_3216Metric_Pad1.30x1.75mm_HandSolder -> Resistor_SMD:R_0603_1608Metric
- R20, R21, R5, R6: footprint Resistor_SMD:R_1206_3216Metric_Pad1.30x1.75mm_HandSolder -> Resistor_SMD:R_0603_1608Metric
- U1: value PI3B3253LEX -> PI3B3253LE; Manufacturer_Part_Number PI3B3253LEX -> PI3B3253LE; Mouser Part (none) -> 729-PI3B3253LE; Mouser Part Number 729-PI3B3253LEX -> (none); Mouser Price/Stock https://www.mouser.co.uk/ProductDetail/Diodes-Incorporated/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 -> https://www.mouser.com/ProductDetail/729-PI3B3253LE
Connections:
- net +3.3V: now also R3.2, R4.1
- net AMP_Vn: now also C44.2, U7.5 (VOUT), IC1.4 (-VS), IC2.4 (-VS)
- net GND: now also R16.1, C45.1, C46.1, IC1.5 (REF), IC2.5 (REF), R23.2, R24.1, R25.2, U8.2 (GND), U8.3 (GND), U8.6 (GND), U8.7 (GND)
- net IA0: now also R16.2, IC1.2 (-IN)
- net IA1: now also IC2.2 (-IN), R24.2
- net IA2: now also IC2.3 (+IN), R25.1
- net IA3: now also IC1.3 (+IN), R23.1
- net SCL: now also R3.1
- net SDA: now also R4.2
- net at C29.2, PS1.5 (VOUT): now also C43.2, U7.2 (VIN), U7.3 (EN)
- net AMP_Vp: now reaches PS1.1 ((N.C.)_BOOST)
- net AMP_Vp: now also C42.1, C7.1, C9.1, PS1.8 (V+), C46.2, IC1.7 (+VS), IC2.7 (+VS), U8.1 (OUT)
- net at FB4.1: now also C40.2, U1.7 (YA), U1.9 (YB); no longer R16.2
- net at J2.2: now also IC1.6 (OUT)
- net at J2.3: now also IC2.6 (OUT)
- net at U6.10 (CLK0): now also C41.1
- net I_GS1: no longer names the net of R1.1
- net I_GS1: now also IC1.1 (RG_1)
- net I_GS2: no longer names the net of R1.2
- net I_GS2: now also IC1.8 (RG_2)
- net LO_CLK: no longer names the net of U6.9 (CLK1)
- net LO_CLK: no longer C41.1
- net Q_GS1: no longer names the net of R2.1
- net Q_GS1: now also IC2.1 (RG_1)
- net Q_GS2: no longer names the net of R2.2
- net Q_GS2: now also IC2.8 (RG_2)
- removed net TAYLOE_IN: C40.2, R16.1, U1.7 (YA), U1.9 (YB)
- net VBUS: no longer names the net of C31.1, U4.1 (VIN), U4.3 (EN)
- net VBUS: now also J4.2 (Pin_2), C45.2, U8.8 (IN); no longer C7.1, C9.1
- no-connect marks 16 -> 6
Other:
- note added: "+30v in MAX!!!!! (minimum 10 please thanks)"
- note added: "check sampl cap values"
- note added: "ground pour!!!"
- moved on the sheet: C1, C10, C11, C12, C14, C2, C29, C3, C31, C32, C33, C34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

Commit message: save
Parts:
- removed C41: 0.1u, Capacitor_SMD:C_0603_1608Metric, symbol Device:C_Small
- removed R20, R21: 10k, Resistor_SMD:R_0603_1608Metric, symbol Device:R_Small
- removed U1: PI3B3253LE, Package_SO:TSSOP-16_4.4x5mm_P0.65mm, symbol tayloe:PI3B3253LEX
- added FB5: 330R/0.5A, Inductor_SMD:L_0603_1608Metric, symbol Device:FerriteBead_Small
- added U1: SN74CBTLV3253PWR, Package_SO:TSSOP-16_4.4x5mm_P0.65mm, symbol tayloe:SN74CBTLV3253PWR
- C2: value 0.1u -> 0.47u
Connections:
- net +3.3V: now also FB5.1; no longer C2.2
- net CLKIN: now also U6.10 (CLK0); no longer U2.3 (1CLK)
- net GND: now also C2.2, U1.1 (1~{OE}), U1.15 (2~{OE}), U1.8 (GND); no longer C2.1
- net IA0: now also U1.10 (2B1), U1.6 (1B1)
- net IA1: now also U1.11 (2B2), U1.5 (1B2)
- net IA2: now also U1.12 (2B3), U1.4 (1B3)
- net IA3: now also U1.13 (2B4), U1.3 (1B4)
- net S0: now also U1.14 (S0)
- net S1: now also U1.2 (S1)
- net at C40.2, FB4.1: now also U1.7 (1A), U1.9 (2A)
- new net: C2.1, FB5.2, U1.16 (VCC)
Other:
- note removed: "ground pour!!!"
- moved on the sheet: C38, C39, R3, R4, U6, Y2

Commit message: rev 3
Parts:
- removed C12: 47u, Capacitor_SMD:CP_Elec_5x5.3, symbol Device:C_Polarized_Small
- removed C14, C29: 22u, Capacitor_SMD:CP_Elec_5x5.3, symbol Device:C_Polarized_Small
- removed C38, C39, C46, C7, C9: 0.1u, Capacitor_SMD:C_0603_1608Metric, symbol Device:C_Small
- removed C42: 0.1u, Capacitor_SMD:CP_Elec_5x5.3, symbol Device:C_Polarized_Small
- removed C43, C44: 4.7u, Capacitor_SMD:C_0603_1608Metric, symbol Device:C_Small
- removed C45: 0.33u, Capacitor_SMD:C_0603_1608Metric, symbol Device:C_Small
- removed IC1, IC2: INA828IDR, Package_SO:SOIC-8_3.9x4.9mm_P1.27mm, symbol tayloe:INA828IDR
- removed J4: Conn_01x02_Pin, Connector_PinHeader_2.54mm:PinHeader_1x02_P2.54mm_Vertical, symbol Connector:Conn_01x02_Pin
- removed PS1: MAX1044CPA+, tayloe:DIP794W56P254L938H457Q8N, symbol tayloe:MAX1044CPA+
- removed R16, R23, R24, R25: 47k, Resistor_SMD:R_0603_1608Metric, symbol Device:R_Small
- removed R5: 4.02k, Resistor_SMD:R_0603_1608Metric, symbol Device:R_Small
- removed R6: 1k, Resistor_SMD:R_0603_1608Metric, symbol Device:R_Small
- removed U7: ADP7182AUJZ-5.0, Package_TO_SOT_SMD:TSOT-23-5, symbol Regulator_Linear:ADP7182AUJZ-5.0
- removed U8: L78L08_SO8, Package_SO:SOIC-8_3.9x4.9mm_P1.27mm, symbol Regulator_Linear:L78L08_SO8
- added C12: 0.47u, Capacitor_SMD:C_0603_1608Metric, symbol Device:C_Small
- added C14, C29: 22u, Capacitor_SMD:C_0603_1608Metric, symbol Device:C_Small
- added L3, L4: 10u, Inductor_SMD:L_0603_1608Metric, symbol Device:L_Small
- added U7: ADA4084-2ACPZ-R7, Package_CSP:LFCSP-8-1EP_3x3mm_P0.5mm_EP1.6x2.34mm_ThermalVias, symbol tayloe:ADA4084-2ACPZ-R7
- C11: value 0.1u -> 22u
- FB4: value 600R/0.5A -> 330R/0.5A; Mouser Part 81-BLM18HK601SN1D -> 81-BLM18HK331SN1
- R1, R2: value 330 -> 1k; Mouser Part 603-RT0603DRE07330RL -> (none)
Connections:
- net +3.3V: now also R1.1, L3.1, L4.1; no longer U6.1 (VDD), U6.7 (VDDO)
- net AMP_Vp: now also C29.1, L4.2, U7.8 (V+)
- net CLKIN: now also U2.3 (1CLK)
- net GND: now also R2.1, C12.2, C14.2, C29.2, U7.4 (V-), U7.9 (EP); no longer C10.2, C8.2
- net IA0: now also U7.2 (-IN_A)
- net IA1: now also U7.6 (-IN_B)
- net IA2: now also U7.5 (+IN_B)
- net IA3: now also U7.3 (+IN_A)
- net at J2.3: now also C8.1
- net at R2.2: now also C11.1, FB4.1, R1.2
- net VBUS: now reaches C31.1, U4.1 (VIN), U4.3 (EN)
- net at FB4.2: now also C40.2, U1.7 (1A), U1.9 (2A), C12.1; no longer C11.1
- net at J2.2: now also C10.2
- net AMP_Vn: no longer names the net of C10.1
- net AMP_Vn: now also U7.7 (OUT_B); no longer C8.1
- new net: C14.1, L3.2, U6.1 (VDD), U6.7 (VDDO)
- new net: C8.2, U7.1 (OUT_A)
- no-connect marks 6 -> 4
Other:
- note removed: "+30v in MAX!!!!! (minimum 10 please thanks)"
- note removed: "I Channel"
- note removed: "Q Channel"
- moved on the sheet: C3, C31, C32, C4, C5, C6, U4

Commit message: rev 3.1
Parts:
- added C7, C9: 670p, Capacitor_SMD:C_0603_1608Metric, symbol Device:C_Small
- added R12, R13, R5, R6: 100, Resistor_SMD:R_0603_1608Metric, symbol Device:R_Small
- added R14, R15: 10k, Resistor_SMD:R_0603_1608Metric, symbol Device:R_Small
Connections:
- net IA0: now also R5.1; no longer U7.2 (-IN_A)
- net IA1: now also R12.2; no longer U7.6 (-IN_B)
- net IA2: now also R13.1; no longer U7.5 (+IN_B)
- net IA3: now also R6.2; no longer U7.3 (+IN_A)
- net at C10.1, U7.7 (OUT_B): now also C9.1, R15.2
- net at C8.2, U7.1 (OUT_A): now also C7.2, R14.2
- net at C8.1, J2.3: now also J2.4
- new net: C7.1, R14.1, R5.2, U7.2 (-IN_A)
- new net: R6.1, U7.3 (+IN_A)
- new net: R13.2, U7.5 (+IN_B)
- new net: C9.2, R12.1, R15.1, U7.6 (-IN_B)
Other:
- moved on the sheet: C10, C29, C31, C32, C5, C6, C8, J2, L4, U4, U7
